File: tests_nov24/control.kicad_sch (KiCad schematic)
At the start: 0 parts

Commit message: Control, DC-DC and motor
Parts:
- added D1: LED, symbol Device:LED
- added Q1: NPN, symbol Simulation_SPICE:NPN
- added R3, R4, R5: R, symbol Device:R
- added SW3: SW_Push, symbol Switch:SW_Push
- added U1: ~, symbol Exocet_Tests:TS0010D-Relay_Board
- added U2: STM32G474RBTx, Package_QFP:LQFP-64_10x10mm_P0.5mm, symbol MCU_ST_STM32G4:STM32G474RBTx
Connections:
- new net: D1.2 (A), R5.1
- new net: R3.2, SW3.2, U2.2 (PC13)
- new net: R4.1, U2.19 (PA5)
- new net: Q1.2 (B), R4.2
- new net: U1. (~{IN_2}), U2.12 (PA0)
- new net: U1. (~{IN_2}), U2.13 (PA1)
- new net: D1.1 (K), Q1.1 (C)
- new net +24V: U1. (~{IN_2})
- new net +3.3V: R5.2, SW3.1, U1. (~{IN_2}), U2.16 (VDD), U2.32 (VDD), U2.48 (VDD), U2.64 (VDD)
- new net +5V: U1. (~{IN_2})
- new net Charge level 2: U1. (~{IN_2})
- new net GND: Q1.3 (E), R3.1, U1. (~{IN_2}), U2.15 (VSS), U2.31 (VSS), U2.47 (VSS), U2.63 (VSS)
- new net Source isolation: U1. (~{IN_2})
- new net ~{Source isolation}: U1. (~{IN_2})
- no-connect marks 0 -> 2
