File: tests_nov24/tests_nov24.kicad_sch (KiCad schematic)
At the start: 0 parts

Commit message: First draft or relay layout
Parts:
- added BT1, BT2: EWLI-48V5120, symbol Device:Battery
- added F1, F2: Fuse, symbol Device:Fuse
- added K1, K2, K3: Relay_SPST-NO, symbol Relay:Relay_SPST-NO
- added K4, K5: Relay board, symbol Relay:Relay_SPDT
- added R1, R2: R, symbol Device:R
- added SW1: E-Stop NC, symbol Switch:SW_Push_Open
- added SW2: E-Stop NO, symbol Switch:SW_Push
Connections:
- new net: K2.14, R1.2
- new net: K1.14, K2.13, K3.13, R2.1
- new net: BT1.1 (+), F1.2
- new net: K1.A2, SW1.2 (B)
- new net: BT2.1 (+), F2.2
- new net +24V: K4.11, K5.11, SW2.1
- new net +48V: F1.1, F2.1, K1.13
- new net Charge level 2: K3.A2, K5.14
- new net Charge level 2 control: K5.A2
- new net DC-DC A+: K3.14, R2.2
- new net GND: BT1.2 (-), BT2.2 (-), K1.A1, K2.A1, K3.A1, K4.A1, K5.A1, R1.1
- new net Source isolation: K4.14, SW1.1 (A)
- new net Source isolation control: K4.A2
- new net ~{Source isolation}: K2.A2, K4.12, SW2.2
- no-connect marks 0 -> 1
Other:
- added sheet Control (control.kicad_sch)

Commit message: Control, DC-DC and motor
Parts:
- removed K4, K5: Relay board, symbol Relay:Relay_SPDT
- added F3: Fuse, symbol Device:Fuse
- added SW4: SW_Push, symbol Switch:SW_Push
- added U3: ~, symbol Exocet_Tests:Brightloop_BB-MP
- added U4: ~, symbol Exocet_Tests:Outdrive_5.0
- added U5: ~, symbol Exocet_Tests:RDT_Throttle
- BT1, BT2: value EWLI-48V5120 -> 48V
- F1, F2: value Fuse -> 60A
- K1: value Relay_SPST-NO -> Source Isolation Contactor
- K2: value Relay_SPST-NO -> Discharge Contactor
- K3: value Relay_SPST-NO -> Charge Contactor
- R1, R2: value R -> 50W, 180Ω
Connections:
- net DC-DC A+: now also U3. (B-)
- net GND: now also U3. (B-)
- new net: U4. (Throttle_Sig), U5. (Sig) (x3)
- new net: F3.1, U3. (B-)
- new net: F3.2, SW4.1
- new net: SW4.2, U4. (Throttle_Sig)
- new net: U3. (B-), U4. (Throttle_Sig)
- no-connect marks 1 -> 6
Other:
- moved on the sheet: BT1, BT2, F1, F2
