File: electrical-layout/h2_control.kicad_sch (KiCad schematic)
At the start: 5 parts, among them U10 SPDX???, U11 SPDX???, U12 ??, U13 ??, U9 PCB02

Commit message: layout-2025: change to version 3.0
A few changes were made for this new version:
- Version and dates were changed on all sheets
- Added a switch (temporary symbol) after the telemetry battery
- A few notes were removed, as these have either been resolved or
discussed somewhere else
- Changed battery symbol to multi-cell battery
Other:
- title: H2 Control Plate -> H2 Control
Changed lines of the file:
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@@
 	(paper "A4")
 	(title_block
-		(title "H2 Control Plate")
-		(date "2025-07-17")
-		(rev "v0.1.0")
+		(title "H2 Control")
+		(date "2025-09-06")
+		(rev "v0.3.0")
 	)
 	(text_box "Rename these to be more descriptive (i.e. High Pressure Valve Actuator)"
