File: electrical-layout/h2_control.kicad_sch (KiCad schematic)
At the start: 5 parts, among them U10 SPDX???, U11 SPDX???, U12 ??, U13 ??, U9 PCB02

Commit message: layout-2025: update many parts of the layout
What a goooood commit message!

... sorry
Parts:
- removed U10, U11: SPDX???, symbol Exocet:Hanbay_Valve_Actuator
- removed U12, U13: ??, symbol Exocet:Swagelok_Manometer
- removed U9: PCB02, symbol Exocet:H2_Control_Pcb
Connections:
- no-connect marks 6 -> 0
