File: electrical-layout/electrical-layout.kicad_sch (KiCad schematic)
At the start: 0 parts

Commit message: layout-2025: update many parts of the layout
What a goooood commit message!

... sorry
Other:
- removed sheet H2 Control
- sheet Cockpit ports: added DMS, ESTOP, MOTOR_THROTTLE; removed none
- sheet Control Box ports: added BOP+, DMS, ESTOP, HV_BUS+, HV_BUS-, MOTOR_SIGNALS, MOTOR_THROTTLE; removed none
- sheet Power System ports: added AUXILIARY_BATT-, AUXILIARY_BATT_CTL, AUXILIARY_SHUNT+, AUXILIARY_SHUNT-, BOP+, BOP_SWITCH_CTL, BRAKE_RESISTOR_CTL, CHARGE_CTLR_CTL, CHARGE_CTLR_UART, DCDC_PRECHARGE_STG1, DCDC_PRECHARGE_STG2, FC_USB, HV_BUS+, HV_BUS-, IMD_SIG, MOTOR_PRECHARGE_STG1, MOTOR_PRECHARGE_STG2, MOTOR_SIGNALS, STORAGE_BATT-, STORAGE_BATT_CTL, STORAGE_SHUNT+, STORAGE_SHUNT-; removed CAN
