File: electrical-layout/cockpit.kicad_sch (KiCad schematic)
At the start: 10 parts, among them SW2 Start Button, SW3 Stop Button, SW4 Dead Man's Switch, SW6 Emergency Stop Button, U5 PCB Cockpit, U6 Raspberry Pi 4B+, U7 Pilot Display, U8 Arduino MKR NB 1500

Commit message: layout-2025: update many parts of the layout
What a goooood commit message!

... sorry
Parts:
- removed U6: Raspberry Pi 4B+, symbol Exocet:Display_Controller
- removed U8: Arduino MKR NB 1500, symbol Exocet:Telemetry_Transmitter
- added D1: Misc Status LED, symbol Device:LED
- added J1: M12 Connector, symbol Exocet:M12_Connector
- added M1: RPi CPU Fan, symbol Exocet:Fan_3pin_PWM
- added SW1: Extra Button, symbol Switch:SW_Push
- added U16: RPi CAN Hat, symbol Exocet:RPi_CAN_Hat
- added U17: Sensors PCB, symbol Exocet:Sensors_PCB
- added U2: Connection PCB, symbol Exocet:Connection_PCB
- added U23: Motor Throttle, symbol Exocet:Motor_Throttle
- added U6: Raspberry Pi 4B+, symbol Exocet:Raspberry_Pi
- added U8: GPS Antenna, symbol Exocet:GPS_Antenna
- SW6: DIST (none) -> Future Electronics; MFR (none) -> Harting; MPN (none) -> 09454530100
- U5: value PCB Cockpit -> Cockpit PCB; DIST (none) -> JLCPCB; MFR (none) -> Exocet; MPN (none) -> PCB01
- U7: DIST (none) -> Waveshare; MFR (none) -> Waveshare; MPN (none) -> 5inch HDMI LCD (G)
Connections:
- net DMS+: no longer names the net of SW4.1
- net DMS-: no longer names the net of SW4.2
- net ESTOP+: no longer names the net of SW6.1 (A)
- net ESTOP-: no longer names the net of SW6.2 (B)
- new net: U6. (HDMI), U7. (HDMI)
- new net: U16. (GPIO), U6. (HDMI)
- new net: D1.1 (K), U5. (LED3-)
- new net: D1.2 (A), U5. (LED3-)
- new net: SW1.1, U5. (LED3-)
- new net: SW1.2, U5. (LED3-)
- new net: M1. (-), U16. (GPIO) (x3)
- new net Earth: U2. (GND)
- now unconnected: U7. (HDMI)

Commit message: layout-2025: add power breadboard and connections
Parts:
- removed M1: RPi CPU Fan, symbol Exocet:Fan_3pin_PWM
- removed U17: Sensors PCB, symbol Exocet:Sensors_PCB
- removed U8: GPS Antenna, symbol Exocet:GPS_Antenna
Connections:
- net Earth is gone; now on net Frame: U2. (GND)
- net at U16. (GPIO): no longer U6. (HDMI)
- net Frame: now reaches U2. (GND)
- now unconnected: U16. (GPIO), U16. (GPIO), U16. (GPIO)
- no-connect marks 4 -> 12
